File: MOSFET_CTL_BRD/mosfet_ctl.sch (EAGLE design)
At the start: 245 parts, among them IC1 MCP23008, IC10 ACS712, IC11 MCP23008, IC12 MCP23008, IC13 MCP2518, IC14 MCP2562FD, IC15 4051, IC16 4051, IC18 LMR50410, IC2 ATMEGA328PTQFP, IC3 ACS712, IC4 ACS712, IC5 ACS712, IC6 ACS712, IC7 ACS712, IC8 ACS712, IC9 ACS712, Q10 SIRA80DP-T1-RE3, Q11 BC857, Q12 SIRA80DP-T1-RE3, Q13 BC857, Q14 SIRA80DP-T1-RE3, Q15 BC857, Q16 SIRA80DP-T1-RE3, Q17 BC857, Q18 SIRA80DP-T1-RE3, Q19 BC857, Q20 SIRA80DP-T1-RE3, Q5 BC857, Q6 SIRA80DP-T1-RE3, Q7 BC857, Q8 SIRA80DP-T1-RE3, Q9 BC857, X10 KEYSTONE_7800, X11 KEYSTONE_7800, X12 KEYSTONE_7800, X13 KEYSTONE_7800, X14 KEYSTONE_7800, X15 KEYSTONE_7800, X16 KEYSTONE_7800, X17 KEYSTONE_7800, X18 KEYSTONE_7800, X19 KEYSTONE_7800, X20 KEYSTONE_7800, X21 KEYSTONE_7800, X22 KEYSTONE_7800, X23 KEYSTONE_7800, X24 KEYSTONE_7800, X25 KEYSTONE_7800, X26 KEYSTONE_7800, X27 KEYSTONE_7800, X28 KEYSTONE_7800, X29 KEYSTONE_7800, X3 RJ11-4RJ11-4, X30 KEYSTONE_7800, X31 KEYSTONE_7800, X32 KEYSTONE_7800, X33 KEYSTONE_7800, X34 KEYSTONE_7800, X35 KEYSTONE_7800, X36 KEYSTONE_7800, X37 KEYSTONE_7800, X38 KEYSTONE_7800, X39 KEYSTONE_7800, X4 RJ11-4RJ11-4, X40 KEYSTONE_7800, X9 KEYSTONE_7800

Commit message: Layout updates for MOSFET & LIGHTING boards. Add new boards REMOTE_SWITCH, CAPACITIVE_SWITCH, VANBUS_HUB
Parts:
- removed C36, C37, C39: 100n, SMD:CAPACITOR0805
- removed C38: 10u, SMD:CAPACITOR1206
- removed D39: 1N4148, SMD:DIODESOD-123
- removed D40: TVS 15V, SMD:DIODE_ZENERDO-214AC
- removed F10, F9: 30A, THT:KEYSTONE-3557-2
- removed IC18: LMR50410, SMD:LMR50410
- removed OK10, OK9: TLP290, SMD:OPTOCOUPLERSO4
- removed Q17, Q19: BC857, SMD:TRANSISTOR_PNPSOT23-CBE
- removed Q18, Q20: SIRA80DP-T1-RE3, SMD:MOSFET_N_CHANNELPPAKSO8
- removed R70: 2k2, SMD:RESISTOR0805
- removed R71: 22k1, SMD:RESISTOR0805
- removed XTAL4: 40MHz, SMD:CRYSTAL_GND5X3.2
- added C27, C28, C29, C30: 100n, SMD:CAPACITOR0805
- added D7: 1N4148, SMD:DIODESOD-123
- added D8: RED, SMD:LED1206
- added F1, F2: 30A, THT:KEYSTONE-3557-2
- added IC17: MCP2562FD, SMD:MCP2562FDSO08
- added OK1, OK2: TLP290, SMD:OPTOCOUPLERSO4
- added Q1, Q3: SIRA80DP-T1-RE3, SMD:MOSFET_N_CHANNELPPAKSO8
- added Q2, Q4: BC857, SMD:TRANSISTOR_PNPSOT23-CBE
- added R13: 16k, SMD:RESISTOR0805
- added R9: 1k, SMD:RESISTOR0805
- added XTAL1: 16MHz, SMD:CRYSTAL_GND5X3.2
- C1, C11, C13, C15, C3, C5, C7, C9: value 100n -> 1n
- C10, C12, C14, C16, C18, C6, C8: value 1n -> 100n
- C17: value 100n -> 10u; device SMD:CAPACITOR0805 -> SMD:CAPACITOR1206
- C19: value 100n -> 22p
- C20: value 1n -> 22p
- C21: value 100n -> 1u
- C24: value 22p -> 10u; device SMD:CAPACITOR0805 -> SMD:CAPACITOR1206
- C25: value 22p -> 100n
- C26: value 1u -> 100n
- C31: value 10u -> 100n; device SMD:CAPACITOR1206 -> SMD:CAPACITOR0805
- D1, D13, D9: value RED -> TVS 15V; device SMD:LED1206 -> SMD:DIODE_ZENERDO-214AC
- D12, D16, D36: value TVS 15V -> RED; device SMD:DIODE_ZENERDO-214AC -> SMD:LED1206
- D18, D22, D26, D30, D34: value GREEN -> 1N4148; device SMD:LED1206 -> SMD:DIODESOD-123
- D19, D23, D27, D31, D35, D6: value 1N4148 -> GREEN; device SMD:DIODESOD-123 -> SMD:LED1206
- D3: value AMBER -> 1N4148; device SMD:LED1206 -> SMD:DIODESOD-123
- D33: value RED -> 1N4148; device SMD:LED1206 -> SMD:DIODESOD-123
- D37: value RED -> AMBER
- D38: value GREEN -> AMBER
- D4: value AMBER -> RED
- D5: value 1N4148 -> TVS 15V; device SMD:DIODESOD-123 -> SMD:DIODE_ZENERDO-214AC
- H1, H2, H3, H4: value MOUNT-PAD-ROUND3.0 -> MOUNT-PAD-ROUND3.2; device holes:MOUNT-PAD-ROUND3.0 -> THT:MOUNT-PAD-ROUND3.2
- IC1: value MCP23008 -> ACS712; device SMD:MCP23008SO18W -> SMD:ACS712
- IC10: value ACS712 -> LMR50410; device SMD:ACS712 -> SMD:LMR50410
- IC12: value MCP23008 -> 4051; device SMD:MCP23008SO18W -> SMD:4051SO16
- IC13: value MCP2518 -> 4051; device SMD:MCP2518FDSO14 -> SMD:4051SO16
- IC14: value MCP2562FD -> MCP23008; device SMD:MCP2562FDSO08 -> SMD:MCP23008SO18W
- IC15: value 4051 -> MCP23008; device SMD:4051SO16 -> SMD:MCP23008SO18W
- IC16: value 4051 -> MCP2518; device SMD:4051SO16 -> SMD:MCP2518FDSO14
- IC2: value ATMEGA328PTQFP -> ACS712; device SMD:ATMEGA328PTQFP -> SMD:ACS712
- IC9: value ACS712 -> ATMEGA328PTQFP; device SMD:ACS712 -> SMD:ATMEGA328PTQFP
- Q5, Q7: value BC857 -> SIRA80DP-T1-RE3; device SMD:TRANSISTOR_PNPSOT23-CBE -> SMD:MOSFET_N_CHANNELPPAKSO8
- Q6, Q8: value SIRA80DP-T1-RE3 -> BC857; device SMD:MOSFET_N_CHANNELPPAKSO8 -> SMD:TRANSISTOR_PNPSOT23-CBE
- R1, R15, R22, R35, R42, R49, R56: value 2k2 -> 1k
- R10: value 470 -> 2k2
- R11: value 470 -> 1k
- R12: value 120 -> 33k
- R14: value 88k7 -> 2k2
- R16, R23: value 33k -> 1k
- R17, R24, R59, R66: value 16k -> 2k2
- R19, R26: value 1k -> 33k
- R2, R4, R8: value 10k -> 1k
- R20, R27: value 1k -> 16k
- R30, R37, R44, R51: value 33k -> 16k
- R31, R38, R45, R52: value 16k -> 33k
- R33, R40, R47, R54: value 1k -> 2k2
- R5: value 2k2 -> 33k
- R57, R63, R64: value 2k2 -> 10k
- R58, R65: value 33k -> 2k2
- R6: value 2k2 -> 16k
- R60: value 1k -> 88k7
- R61: value 1k -> 22k1
- R62: value 1k -> 10k
- R67, R68: value 1k -> 470
- R69: value 1k -> 120
- R7: value 10k -> 2k2
- S1: value 219-08 -> TACTILE_SWITCH6.2MM; device switch-dil:219-08 -> SMD:TACTILE_SWITCH6.2MM
- S10: value TACTILE_SWITCH6.2MM -> SWITCH_DIL08; device SMD:TACTILE_SWITCH6.2MM -> SMD:SWITCH_DIL08
- X3, X4: value RJ11-4RJ11-4 -> RJ11-4HORIZ; device THT:RJ11-4RJ11-4 -> THT:RJ11-4HORIZ
- XTAL2: value 16MHz -> 40MHz
- renumbered JP3 to X1, JP4 to X2, JP6 to JP1, L2 to L1
Connections:
- removed net N$111 (its old number): D37.C, Q19.E
- removed net N$113 (its old number): Q19.C, R64.2
- removed net N$119 (its old number): OK10.EMIT, Q20.G, R69.2
- removed net N$39 (its old number): D13.C, Q7.E
- removed net N$41 (its old number): Q7.C, R22.2
- removed net N$47 (its old number): OK4.EMIT, Q8.G, R27.2
- removed net N$74 (its old number): D27.A, F7.2, IC7.I+
- new net N$26: D3.A, F1.2, IC1.I+
- new net N$51: D8.C, Q4.E
- new net N$53: Q4.C, R14.2
- new net N$59: OK2.EMIT, Q3.G, R8.2
- new net N$75: D12.C, Q6.E
- new net N$77: Q6.C, R21.2
- new net N$83: OK3.EMIT, Q5.G, R15.2
- net +12V: now also C24.1, C25.1, IC10.EN, IC10.VIN; no longer C31.1, C37.1, IC18.EN, IC18.VIN
- net ADC_MUX_A: now also IC12.A, IC13.A, IC9.PD5(T1); no longer IC15.A, IC16.A, IC2.PD5(T1)
- net ADC_MUX_B: now also IC12.B, IC13.B, IC9.PD6(AIN0); no longer IC15.B, IC16.B, IC2.PD6(AIN0)
- net ADC_MUX_C: now also IC12.C, IC13.C, IC9.PD7(AIN1); no longer IC15.C, IC16.C, IC2.PD7(AIN1)
- net GND: now also C1.2, C2.2, C22.1, C26.1, C27.2, C28.2, C29.1, C30.1, C35.1, D35.C, D36.C, IC12.VEE, IC13.VEE, IC14.A0, IC14.A1, IC14.A2, IC15.A2, IC17.GND, IC17.STBY, IC2.GND, IC9.AGND, IC9.GND@3, IC9.GND@5, OK1.C, OK2.C, Q1.S, Q3.S, Q5.S, Q7.S, R1.1, R13.1, R14.1, R21.1, R28.1, R30.1, R37.1, R44.1, R51.1, R6.1, R61.1, R7.1, R8.1, S1.1, S10.10, S10.11, S10.12, S10.13, S10.14, S10.15, S10.16, S10.9, XTAL1.2; no longer C1.1, C2.1, C21.1, C22.2, C23.2, C35.2, C36.1, C37.2, C38.1, D1.C, D2.C, IC1.A1, IC1.A2, IC11.A0, IC12.A2, IC14.STBY, IC15.VEE, IC16.VEE, IC18.GND, IC2.AGND, IC2.GND@3, IC2.GND@5, IC9.GND, OK10.C, OK9.C, Q18.S, Q20.S, Q6.S, Q8.S, R17.1, R24.1, R31.1, R38.1, R45.1, R52.1, R57.1, R59.1, R62.1, R64.1, R66.1, R69.1, R71.1, S1.10, S1.11, S1.12, S1.13, S1.14, S1.15, S1.16, S1.9, S10.1, XTAL4.2
- net I2C_SCL: now also IC14.SCL, IC15.SCL, IC9.PC5(ADC5/SCL), R58.1; no longer IC1.SCL, IC12.SCL, IC2.PC5(ADC5/SCL), R6.1
- net I2C_SDA: now also IC14.SDA, IC15.SDA, IC9.PC4(ADC4/SDA), R59.2; no longer IC1.SDA, IC12.SDA, IC2.PC4(ADC4/SDA), R5.2
- net INT_BTN: now also D33.C, D34.C, IC9.PD2(INT0); no longer D5.C, D6.C, IC2.PD2(INT0)
- net INT_CAN: now also IC16.INT, IC9.PD3(INT1); no longer IC13.INT, IC2.PD3(INT1)
- net IV_OUT_A: now also IC13.X, IC9.PC0(ADC0); no longer IC16.X, IC2.PC0(ADC0)
- net IV_OUT_B: now also IC12.X, IC9.PC1(ADC1); no longer IC15.X, IC2.PC1(ADC1)
- net I_OUT_1: now also IC1.VI_OUT, IC12.X0; no longer IC15.X0, IC3.VI_OUT
- net I_OUT_2: now also IC12.X2, IC2.VI_OUT; no longer IC15.X2, IC5.VI_OUT
- net I_OUT_3: now also IC12.X6, IC3.VI_OUT; no longer IC15.X6, IC7.VI_OUT
- net I_OUT_4: now also IC12.X5, IC4.VI_OUT; no longer IC15.X5, IC9.VI_OUT
- net I_OUT_5: now also IC13.X4, IC5.VI_OUT; no longer IC10.VI_OUT, IC16.X4
- net I_OUT_6: now also IC13.X7, IC6.VI_OUT; no longer IC16.X7, IC8.VI_OUT
- net I_OUT_7: now also IC13.X3, IC7.VI_OUT; no longer IC16.X3, IC6.VI_OUT
- net I_OUT_8: now also IC13.X1, IC8.VI_OUT; no longer IC16.X1, IC4.VI_OUT
- net LED: now also IC9.PB0(ICP), R66.2; no longer IC2.PB0(ICP), R1.2
- net MOSFET_1: now also IC14.GPIO4, R2.1; no longer IC11.GPIO4, R18.1
- net MOSFET_2: now also IC14.GPIO5, R9.1; no longer IC11.GPIO5, R32.1
- net MOSFET_3: now also IC14.GPIO6, R16.1; no longer IC11.GPIO6, R46.1
- net MOSFET_4: now also IC14.GPIO7, R23.1; no longer IC11.GPIO7, R60.1
- net MOSFET_5: now also IC14.GPIO0, R35.1; no longer IC11.GPIO0, R67.1
- net MOSFET_6: now also IC14.GPIO1, R42.1; no longer IC11.GPIO1, R53.1
- net MOSFET_7: now also IC14.GPIO2, R49.1; no longer IC11.GPIO2, R39.1
- net MOSFET_8: now also IC14.GPIO3, R56.1; no longer IC11.GPIO3, R25.1
- net N$1: now also D36.A, R66.1; no longer D1.A, R1.1
- net N$10: now also IC15.GPIO1, S10.2; no longer IC12.GPIO1, S1.2
- net N$100: now also D15.C, Q8.B, R26.2; no longer D35.C, Q17.B, R58.2
- net N$101: now also Q8.C, R28.2; no longer Q17.C, R57.2
- net N$102: now also C7.1, IC4.FILTER; no longer C18.1, IC9.FILTER
- net N$103: now also D14.C, R24.2; no longer D34.C, R63.2
- net N$104: now also OK4.A, R23.2; no longer OK9.A, R60.2
- net N$105: now also OK4.COL, R25.1; no longer OK9.COL, R61.1
- net N$106: now also D13.C, D14.A, IC4.I-, R25.2; no longer D34.A, D36.C, IC9.I-, R61.2
- net N$107: now also OK4.EMIT, Q7.G, R22.2; no longer OK9.EMIT, Q18.G, R62.2
- net N$108: now also D13.A, Q7.D, R24.1; no longer D36.A, Q18.D, R63.1
- net N$109: now also D17.A, F5.1; no longer D37.A, F10.1
- net N$11: now also IC15.GPIO2, S10.3; no longer IC12.GPIO2, S1.3
- net N$110: now also D18.A, F5.2, IC5.I-; no longer D39.A, F10.2, IC10.I-
- net N$112: now also D18.C, Q9.B, R31.2; no longer D39.C, Q19.B, R65.2
- net N$114: now also C9.1, IC5.FILTER; no longer C20.1, IC10.FILTER
- net N$115: now also D19.C, R33.2; no longer D38.C, R70.2
- net N$116: now also OK5.A, R35.2; no longer OK10.A, R67.2
- net N$117: now also OK5.COL, R32.1; no longer OK10.COL, R68.1
- net N$118: now also D19.A, D20.C, IC5.I+, R32.2; no longer D38.A, D40.C, IC10.I+, R68.2
- net N$12: now also IC15.GPIO3, S10.4; no longer IC12.GPIO3, S1.4
- net N$120: now also D20.A, Q10.D, R33.1; no longer D40.A, Q20.D, R70.1
- net N$121: now also IC15.GPIO7, S10.8; no longer IC12.GPIO7, S1.8
- net N$122: now also D33.A, IC11.INT; no longer D6.A, IC1.INT
- net N$123: now also D34.A, IC15.INT; no longer D5.A, IC12.INT
- net N$125: now also C23.2, IC10.SW; no longer C39.2, IC18.SW
- net N$126: now also C23.1, IC10.CB; no longer C39.1, IC18.CB
- net N$127: now also IC10.FB, R60.1, R61.2; no longer IC18.FB, R14.1, R71.2
- net N$13: now also IC15.GPIO4, S10.5; no longer IC12.GPIO4, S1.5
- net N$14: now also IC15.GPIO5, S10.6; no longer IC12.GPIO5, S1.6
- net N$15: now also IC15.GPIO6, S10.7; no longer IC12.GPIO6, S1.7
- net N$16: now also IC17.CANL, R69.1; no longer IC14.CANL, R12.1
- net N$17: now also IC17.CANH; no longer IC14.CANH
- net N$18: now also D37.C, IC16.TXCAN, IC17.TXD; no longer D3.C, IC13.TXCAN, IC14.TXD
- net N$19: now also D38.C, IC16.RXCAN, IC17.RXD; no longer D4.C, IC13.RXCAN, IC14.RXD
- net N$2: now also IC11.A0, R62.1; no longer IC1.A0, R2.1
- net N$20: now also C32.2, IC16.OSC2, XTAL2.1; no longer C33.2, IC13.OSC2, XTAL4.1
- net N$21: now also C33.2, IC16.OSC1, XTAL2.3; no longer C32.2, IC13.OSC1, XTAL4.3
- net N$22: now also D37.A, R67.1; no longer D3.A, R10.1
- net N$23: now also D38.A, R68.1; no longer D4.A, R11.1
- net N$24: now also R69.2; no longer R12.2
- net N$25: now also D4.A, F1.1; no longer D9.A, F3.1
- net N$27: now also D4.C, Q2.E; no longer D9.C, Q5.E
- net N$28: now also D3.C, Q2.B, R5.2; no longer D11.C, Q5.B, R16.2
- net N$29: now also Q2.C, R7.2; no longer Q5.C, R15.2
- net N$3: now also C19.1, IC9.PB6(XTAL1/TOSC1), XTAL1.1; no longer C24.1, IC2.PB6(XTAL1/TOSC1), XTAL2.1
- net N$30: now also C1.1, IC1.FILTER; no longer C6.1, IC3.FILTER
- net N$31: now also D2.C, R3.2; no longer D10.C, R21.2
- net N$32: now also OK1.A, R2.2; no longer OK3.A, R18.2
- net N$33: now also OK1.COL, R4.1; no longer OK3.COL, R19.1
- net N$34: now also D1.C, D2.A, IC1.I-, R4.2; no longer D10.A, D12.C, IC3.I-, R19.2
- net N$35: now also OK1.EMIT, Q1.G, R1.2; no longer OK3.EMIT, Q6.G, R20.2
- net N$36: now also D1.A, Q1.D, R3.1; no longer D12.A, Q6.D, R21.1
- net N$37: now also D29.A, F8.1; no longer D13.A, F4.1
- net N$38: now also D30.A, F8.2, IC8.I-; no longer D15.A, F4.2, IC4.I-
- net N$4: now also C20.1, IC9.PB7(XTAL2/TOSC2), XTAL1.3; no longer C25.1, IC2.PB7(XTAL2/TOSC2), XTAL2.3
- net N$40: now also D30.C, Q15.B, R52.2; no longer D15.C, Q7.B, R23.2
- net N$42: now also C15.1, IC8.FILTER; no longer C8.1, IC4.FILTER
- net N$43: now also D31.C, R54.2; no longer D14.C, R28.2
- net N$44: now also OK8.A, R56.2; no longer OK4.A, R25.2
- net N$45: now also OK8.COL, R53.1; no longer OK4.COL, R26.1
- net N$46: now also D31.A, D32.C, IC8.I+, R53.2; no longer D14.A, D16.C, IC4.I+, R26.2
- net N$48: now also D32.A, Q16.D, R54.1; no longer D16.A, Q8.D, R28.1
- net N$49: now also D8.A, F2.1; no longer D17.A, F5.1
- net N$5: now also D35.A, R65.1; no longer D2.A, R3.1
- net N$50: now also D7.A, F2.2, IC2.I+; no longer D19.A, F5.2, IC5.I+
- net N$52: now also D7.C, Q4.B, R12.2; no longer D19.C, Q9.B, R30.2
- net N$54: now also C3.1, IC2.FILTER; no longer C10.1, IC5.FILTER
- net N$55: now also D6.C, R10.2; no longer D18.C, R35.2
- net N$56: now also OK2.A, R9.2; no longer OK5.A, R32.2
- net N$57: now also OK2.COL, R11.1; no longer OK5.COL, R33.1
- net N$58: now also D5.C, D6.A, IC2.I-, R11.2; no longer D18.A, D20.C, IC5.I-, R33.2
- net N$6: now also C21.1; no longer C26.1
- net N$60: now also D5.A, Q3.D, R10.1; no longer D20.A, Q10.D, R35.1
- net N$61: now also D25.A, F7.1; no longer D21.A, F6.1
- net N$62: now also D26.A, F7.2, IC7.I-; no longer D23.A, F6.2, IC6.I-
- net N$64: now also D26.C, Q13.B, R45.2; no longer D23.C, Q11.B, R37.2
- net N$66: now also C13.1, IC7.FILTER; no longer C12.1, IC6.FILTER
- net N$67: now also D27.C, R47.2; no longer D22.C, R42.2
- net N$68: now also OK7.A, R49.2; no longer OK6.A, R39.2
- net N$69: now also OK7.COL, R46.1; no longer OK6.COL, R40.1
- net N$7: now also IC15.A0, R64.1; no longer IC12.A0, R7.1
- net N$70: now also D27.A, D28.C, IC7.I+, R46.2; no longer D22.A, D24.C, IC6.I+, R40.2
- net N$72: now also D28.A, Q14.D, R47.1; no longer D24.A, Q12.D, R42.1
- net N$73: now also D12.A, F3.1; no longer D25.A, F7.1
- net N$76: now also D11.C, Q6.B, R19.2; no longer D27.C, Q13.B, R44.2
- net N$78: now also C5.1, IC3.FILTER; no longer C14.1, IC7.FILTER
- net N$79: now also D10.C, R17.2; no longer D26.C, R49.2
- net N$8: now also IC15.A1, R63.1; no longer IC12.A1, R8.1
- net N$80: now also OK3.A, R16.2; no longer OK7.A, R46.2
- net N$81: now also OK3.COL, R18.1; no longer OK7.COL, R47.1
- net N$82: now also D10.A, D9.C, IC3.I-, R18.2; no longer D26.A, D28.C, IC7.I-, R47.2
- net N$84: now also D9.A, Q5.D, R17.1; no longer D28.A, Q14.D, R49.1
- net N$85: now also D21.A, F6.1; no longer D29.A, F8.1
- net N$86: now also D22.A, F6.2, IC6.I-; no longer D31.A, F8.2, IC8.I-
- net N$88: now also D22.C, Q11.B, R38.2; no longer D31.C, Q15.B, R51.2
- net N$9: now also IC15.GPIO0, S10.1; no longer IC12.GPIO0, S1.1
- net N$90: now also C11.1, IC6.FILTER; no longer C16.1, IC8.FILTER
- net N$91: now also D23.C, R40.2; no longer D30.C, R56.2
- net N$92: now also OK6.A, R42.2; no longer OK8.A, R53.2
- net N$93: now also OK6.COL, R39.1; no longer OK8.COL, R54.1
- net N$94: now also D23.A, D24.C, IC6.I+, R39.2; no longer D30.A, D32.C, IC8.I+, R54.2
- net N$96: now also D24.A, Q12.D, R40.1; no longer D32.A, Q16.D, R56.1
- net N$97: now also D16.A, F4.1; no longer D33.A, F9.1
- net N$98: now also D15.A, F4.2, IC4.I+; no longer D35.A, F9.2, IC9.I+
- net N$99: now also D16.C, Q8.E; no longer D33.C, Q17.E
- net RESET: now also C21.2, IC14.RESET, IC15.RESET, IC9.PC6(/RESET), R57.1, S9.2; no longer C26.2, IC1.RESET, IC12.RESET, IC2.PC6(/RESET), R4.1, S2.2
- net SPI_CLK: now also IC16.SCK, IC9.PB5(SCK); no longer IC13.SCK, IC2.PB5(SCK)
- net SPI_CS_CAN: now also IC16.CS, IC9.PB2(SS/OC1B); no longer IC13.CS, IC2.PB2(SS/OC1B)
- net SPI_MISO: now also IC16.SDO, IC9.PB4(MISO); no longer IC13.SDO, IC2.PB4(MISO)
- net SPI_MOSI: now also IC16.SDI, IC9.PB3(MOSI/OC2); no longer IC13.SDI, IC2.PB3(MOSI/OC2)
- net SW_1: now also IC11.GPIO7, S1.2; no longer IC1.GPIO7, S3.2
- net SW_2: now also IC11.GPIO6, S2.2; no longer IC1.GPIO6, S5.2
- net SW_3: now also IC11.GPIO5, S3.2; no longer IC1.GPIO5, S7.2
- net SW_4: now also IC11.GPIO4, S4.2; no longer IC1.GPIO4, S9.2
- net SW_5: now also IC11.GPIO3, S5.2; no longer IC1.GPIO3, S10.2
- net SW_6: now also IC11.GPIO2, S6.2; no longer IC1.GPIO2, S8.2
- net SW_7: now also IC11.GPIO1, S7.2; no longer IC1.GPIO1, S6.2
- net SW_8: now also IC11.GPIO0, S8.2; no longer IC1.GPIO0, S4.2
- net UART_RX: now also IC9.PD0(RXD); no longer IC2.PD0(RXD)
- net UART_TX: now also IC9.PD1(TXD); no longer IC2.PD1(TXD)
- net VCC: now also C10.1, C12.1, C14.1, C16.1, C18.1, C2.1, C22.2, C26.2, C27.1, C28.1, C29.2, C30.2, C31.1, C35.2, C6.1, C8.1, IC17.VCC, IC17.VIO, IC2.VCC, IC9.AREF, IC9.AVCC, IC9.VCC@4, IC9.VCC@6, R57.2, R58.2, R59.1, R60.2, R62.2, R63.2, R64.2, R65.2, R67.2, R68.2; no longer C1.2, C11.1, C13.1, C15.1, C19.1, C2.2, C21.2, C22.1, C23.1, C3.1, C35.1, C36.2, C38.2, C5.1, C7.1, C9.1, IC10.VCC, IC14.VIO, IC2.AREF, IC2.AVCC, IC2.VCC@4, IC2.VCC@6, IC9.VCC, R10.2, R11.2, R14.2, R2.2, R3.2, R4.2, R5.1, R6.2, R7.2, R8.2
- net V_OUT_1: now also IC12.X3, R5.1, R6.2; no longer IC15.X3, R16.1, R17.2
- net V_OUT_2: now also IC12.X1, R12.1, R13.2; no longer IC15.X1, R30.1, R31.2
- net V_OUT_3: now also IC12.X4, R19.1, R20.2; no longer IC15.X4, R44.1, R45.2
- net V_OUT_4: now also IC12.X7, R26.1, R27.2; no longer IC15.X7, R58.1, R59.2
- net V_OUT_5: now also IC13.X6, R30.2, R31.1; no longer IC16.X6, R65.1, R66.2
- net V_OUT_6: now also IC13.X5, R37.2, R38.1; no longer IC16.X5, R51.1, R52.2
- net V_OUT_7: now also IC13.X0, R44.2, R45.1; no longer IC16.X0, R37.1, R38.2
- net V_OUT_8: now also IC13.X2, R51.2, R52.1; no longer IC16.X2, R23.1, R24.2
