File: CAPACITIVE_SWITCH_BRD/capacitive_switch.brd (EAGLE design)
At the start: 111.8 x 61 mm, 61 parts, among them IC1 ATMEGA328PTQFP, IC2 AT42QT2160, IC3 MCP2518, IC4 MCP2562FD, IC5 LMR50410, T1 CAPACITIVE_TOUCH, X1 FTDI, X2 ISCP, X3 RJ11-4VERT, X4 RJ11-4VERT

Commit message: v0.1 Production Run Commit - Including GERBER Files
Other:
- outline, holes or cut-outs redrawn
- board text added: "CAPACITIVE_TOUCH_SLIDER_V0.1"
- board text added: "RST"
