File: LIGHTING_CTL_BRD/lighting_ctl.sch (EAGLE design)
At the start: 146 parts, among them IC1 ATMEGA328PTQFP, IC2 MCP23008, IC3 PCA9865TSSOP28, IC4 MCP2518, IC5 MCP2562FD, IC6 LMR50410, X1 RJ11-4RJ11-4, X10 KEYSTONE_7788, X11 KEYSTONE_7788, X12 KEYSTONE_7788, X13 KEYSTONE_7788, X14 KEYSTONE_7788, X15 KEYSTONE_7788, X16 KEYSTONE_7788, X17 KEYSTONE_7788, X18 KEYSTONE_7788, X19 KEYSTONE_7788, X2 RJ11-4RJ11-4, X20 KEYSTONE_7788, X21 KEYSTONE_7788, X22 KEYSTONE_7788, X23 KEYSTONE_7788, X24 KEYSTONE_7788, X25 KEYSTONE_7788, X26 KEYSTONE_7788, X27 KEYSTONE_7788, X28 KEYSTONE_7788, X29 KEYSTONE_7788, X30 KEYSTONE_7788, X35 KEYSTONE_7788, X36 KEYSTONE_7788, X37 KEYSTONE_7788, X38 KEYSTONE_7788, X43 KEYSTONE_7788, X44 KEYSTONE_7788, X45 KEYSTONE_7788, X46 KEYSTONE_7788, X7 KEYSTONE_7788, X8 KEYSTONE_7788, X9 KEYSTONE_7788

Commit message: Layout updates for MOSFET & LIGHTING boards. Add new boards REMOTE_SWITCH, CAPACITIVE_SWITCH, VANBUS_HUB
Parts:
- H1, H2, H3, H4: value MOUNT-PAD-ROUND3.0 -> MOUNT-PAD-ROUND3.2; device holes:MOUNT-PAD-ROUND3.0 -> THT:MOUNT-PAD-ROUND3.2
- X1, X2: value RJ11-4RJ11-4 -> RJ11-4HORIZ; device THT:RJ11-4RJ11-4 -> THT:RJ11-4HORIZ
Connections:
- net N$18: now also D11.C; no longer D12.C
- net N$19: now also D12.C; no longer D11.C
Other:
- moved on the sheet: D11, D12, R39, R40
