File: REMOTE_SWITCH_BRD/remote_switch.brd (EAGLE design)
At the start: 127 x 71.2 mm, 98 parts, among them IC1 MCP23008, IC2 MCP23008, IC3 ATMEGA328PTQFP, IC4 MCP2518, IC5 MCP2562FD, IC6 MCP23008, IC7 LMR50410, X1 FTDI, X2 ISCP, X3 RJ11-4VERT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

Commit message: v0.1 Production Run Commit - Including GERBER Files
Other:
- board size 127 x 71.2 mm -> 127 x 71.1 mm
- board text added: "GND"
- board text added: "LED"
- board text added: "PIN 1"
- board text added: "PIN 2"
- board text added: "PIN 3"
- board text added: "REMOTE_ILLUMINATED_SWITCH_V0.1"
- board text added: "SW"
