File: VANBUS_HUB/hub.brd (EAGLE design)
At the start: 66 x 94 mm, 23 parts, among them X1 RJ11-4VERT, X10 RJ11-4VERT, X11 RJ11-4VERT, X12 RJ11-4VERT, X2 RJ11-4VERT, X3 RJ11-4VERT, X4 RJ11-4VERT, X5 RJ11-4VERT, X6 RJ11-4VERT, X7 RJ11-4VERT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

Commit message: v0.1 Production Run Commit - Including GERBER Files
Parts:
- added D1: (no value), SMD:CHIPLED_1206
- added R3: 120, SMD:R0805
Connections:
- new net N$5: D1.C, R3.1
- net +12V: now also D1.A
- net GND: now also R3.2
Routing:
- net +12V: track 264.7 -> 272.4 mm
- net N$5: track 0.00 -> 4.27 mm
- net N$2: vias 1 -> 0
Other:
- board text added: "VANBUS_HUB_V0.1"
