File: VANBUS_HUB/hub.sch (EAGLE design)
At the start: 23 parts, among them X1 RJ11-4VERT, X10 RJ11-4VERT, X11 RJ11-4VERT, X12 RJ11-4VERT, X2 RJ11-4VERT, X3 RJ11-4VERT, X4 RJ11-4VERT, X5 RJ11-4VERT, X6 RJ11-4VERT, X7 RJ11-4VERT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

Commit message: v0.1 Production Run Commit - Including GERBER Files
Parts:
- added D1: (no value), SMD:LED1206
- added R3: 120, SMD:RESISTOR0805
Connections:
- new net N$5: D1.C, R3.1
- net +12V: now also D1.A
- net GND: now also R3.2
Changed lines of the file:
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@@
 <setting verticaltext="up"/>
 </settings>
-<grid distance="0.1" unitdist="inch" unit="inch" style="lines" multiple="1" display="yes" altdistance="0.01" altunitdist="inch" altunit="inch"/>
+<grid distance="0.1" unitdist="inch" unit="inch" style="lines" multiple="1" display="no" altdistance="0.01" altunitdist="inch" altunit="inch"/>
 <layers>
 <layer number="1" name="Top" color="4" fill="1" visible="no" active="no"/>
@@
 <part name="VDD1" library="supply1" library_urn="urn:adsk.eagle:library:371" deviceset="VDD" device=""/>
 <part name="P+2" library="supply1" library_urn="urn:adsk.eagle:library:371" deviceset="+12V" device=""/>
+<part name="D1" library="SMD" library_urn="urn:adsk.eagle:library:29221540" deviceset="LED" device="1206" package3d_urn="urn:adsk.eagle:package:29221563/3"/>
+<part name="R3" library="SMD" library_urn="urn:adsk.eagle:library:29221540" deviceset="RESISTOR" device="0805" package3d_urn="urn:adsk.eagle:package:29221574/3" value="120"/>
+<part name="P+3" library="supply1" library_urn="urn:adsk.eagle:library:371" deviceset="+12V" device=""/>
+<part name="GND4" library="supply1" library_urn="urn:adsk.eagle:library:371" deviceset="GND" device=""/>
 </parts>
 <sheets>
@@
 <instance part="P+2" gate="1" x="162.56" y="162.56" smashed="yes">
 <attribute name="VALUE" x="160.02" y="157.48" size="1.778" layer="96" rot="R90"/>
+</instance>
+<instance part="D1" gate="G$1" x="203.2" y="157.48" smashed="yes">
+<attribute name="NAME" x="206.756" y="152.908" size="1.778" layer="95" rot="R90"/>
+<attribute name="VALUE" x="208.915" y="152.908" size="1.778" layer="96" rot="R90"/>
+</instance>
+<instance part="R3" gate="G$1" x="203.2" y="147.32" smashed="yes" rot="R270">
+<attribute name="NAME" x="204.6986" y="151.13" size="1.778" layer="95" rot="R270"/>
+<attribute name="VALUE" x="199.898" y="151.13" size="1.778" layer="96" rot="R270"/>
+</instance>
+<instance part="P+3" gate="1" x="203.2" y="162.56" smashed="yes">
+<attribute name="VALUE" x="200.66" y="157.48" size="1.778" layer="96" rot="R90"/>
+</instance>
+<instance part="GND4" gate="1" x="203.2" y="139.7" smashed="yes">
+<attribute name="VALUE" x="200.66" y="137.16" size="1.778" layer="96"/>
 </instance>
 </instances>
@@
 <pinref part="P+2" gate="1" pin="+12V"/>
 </segment>
+<segment>
+<pinref part="D1" gate="G$1" pin="A"/>
+<pinref part="P+3" gate="1" pin="+12V"/>
+</segment>
 </net>
 <net name="GND" class="0">
@@
 <wire x1="127" y1="147.32" x2="127" y2="142.24" width="0.1524" layer="91"/>
 <pinref part="GND3" gate="1" pin="GND"/>
+</segment>
+<segment>
+<pinref part="R3" gate="G$1" pin="2"/>
+<pinref part="GND4" gate="1" pin="GND"/>
 </segment>
 </net>
@@
 </segment>
 </net>
+<net name="N$5" class="0">
+<segment>
+<pinref part="D1" gate="G$1" pin="C"/>
+<pinref part="R3" gate="G$1" pin="1"/>
+</segment>
+</net>
